Commit message: Feat: add omni-direction odometry, can use arg:odom_type to decide a type of odometry: diff or omni

File: localization/OpenBase/ROS/open_base/xacro/main.urdf.xacro (robot description, xacro)
@@ -5,40 +5,58 @@
 >
 	<xacro:include filename="$(find open_base)/xacro/rim.urdf.xacro"/>
+	<xacro:include filename="$(find open_base)/xacro/omni.gazebo.xacro"/>
 	<link name="origin_link"/>
 	<link name="base_link">
-	<inertial>
-		<mass value="0.07862944645"/>
-		<inertia
-			ixx="0.00002035985530754"
-			ixy="0"
-			ixz="0"
-			iyy="0.00002035985530754"
-			iyz="0"
-			izz="0.00003945961663220"
-		/>
-	</inertial>
-	<visual>
-		<geometry>
-			<mesh filename="package://open_base/mesh/base.stl"/>
-		</geometry>
-		<material name="base_material">
-			<color rgba="1 1 1 1"/>
-		</material>
-	</visual>
-	<collision>
-		<geometry>
-			<mesh filename="package://open_base/mesh/base.stl"/>
-		</geometry>
-	</collision>
+		<inertial>
+			<mass value="0.07862944645"/>
+			<inertia
+				ixx="0.00002035985530754" ixy="0" ixz="0" iyy="0.00002035985530754" iyz="0" izz="0.00003945961663220"
+			/>
+		</inertial>
+		<visual>
+			<geometry>
+				<mesh filename="package://open_base/mesh/base.stl"/>
+			</geometry>
+			<material name="base_material">
+				<color rgba="1 1 1 1"/>
+			</material>
+		</visual>
+		<collision>
+			<geometry>
+				<mesh filename="package://open_base/mesh/base.stl"/>
+			</geometry>
+		</collision>
 	</link>
-	<joint
-		name="base_joint"
-		type="fixed"
-	>
+	<joint name="base_joint" type="fixed">
 		<parent link="origin_link" />
 		<child link="base_link" />
-		<origin
-			xyz="0 0 0.01905"
-		/>
+		<origin xyz="0 0 0.01905"/>
+	</joint>
+  <link name="base_scan">
+    <visual>
+      <origin xyz="0 0 0.0" rpy="0 0 0"/>
+      <geometry>
+        <mesh filename="package://turtlebot3_description/meshes/sensors/lds.stl" scale="0.0004 0.0004 0.0004"/>
+      </geometry>
+      <material name="base_material"/>
+    </visual>
+    <collision>
+      <origin xyz="0.015 0 -0.0065" rpy="0 0 0"/>
+      <geometry>
+        <cylinder length="0.0315" radius="0.055"/>
+      </geometry>
+    </collision>
+    <inertial>
+      <mass value="0.0114" />
+      <origin xyz="0 0 0" />
+      <inertia ixx="0.001" ixy="0.0" ixz="0.0"
+               iyy="0.001" iyz="0.0"
+               izz="0.001" />
+    </inertial>
+  </link>
+	<joint name="scan_joint" type="fixed">
+		<parent link="base_link" />
+		<child link="base_scan" />
+		<origin xyz="0 0 0.01905"/>
 	</joint>
 	<xacro:rim_macro

Commit message: Feat: sim 3-wheeled omni odometry, not finish

File: localization/OpenBase/ROS/open_base/xacro/main.urdf.xacro (robot description, xacro)
@@ -1,28 +1,30 @@
 <?xml version="1.0"?>
-<robot
-	xmlns:xacro="http://www.ros.org/wiki/xacro"
-	name="open_base"
->
+<robot name="open_base" xmlns:xacro="http://www.ros.org/wiki/xacro">
 	<xacro:include filename="$(find open_base)/xacro/rim.urdf.xacro"/>
 	<xacro:include filename="$(find open_base)/xacro/omni.gazebo.xacro"/>
+	<xacro:property name="scale" value="7.5"/>
+	<gazebo reference="base_link">
+		<material>Gazebo/White</material>
+	</gazebo>
+	<gazebo reference="base_scan">
+		<material>Gazebo/Black</material>
+	</gazebo>
 	<link name="origin_link"/>
 	<link name="base_link">
 		<inertial>
-			<mass value="0.07862944645"/>
-			<inertia
-				ixx="0.00002035985530754" ixy="0" ixz="0" iyy="0.00002035985530754" iyz="0" izz="0.00003945961663220"
-			/>
+      <mass value="1.0" />
+      <origin xyz="0 0 0" />
+      <inertia ixx="0.45" ixy="0.0" ixz="0.0"
+               iyy="0.45" iyz="0.0"
+               izz="0.45" />
 		</inertial>
 		<visual>
 			<geometry>
-				<mesh filename="package://open_base/mesh/base.stl"/>
+				<mesh filename="package://open_base/mesh/base.stl" scale="${scale} ${scale} ${scale}"/>
 			</geometry>
-			<material name="base_material">
-				<color rgba="1 1 1 1"/>
-			</material>
 		</visual>
 		<collision>
 			<geometry>
-				<mesh filename="package://open_base/mesh/base.stl"/>
+				<mesh filename="package://open_base/mesh/base.stl" scale="${scale} ${scale} ${scale}"/>
 			</geometry>
 		</collision>
@@ -37,7 +39,6 @@
       <origin xyz="0 0 0.0" rpy="0 0 0"/>
       <geometry>
-        <mesh filename="package://turtlebot3_description/meshes/sensors/lds.stl" scale="0.0004 0.0004 0.0004"/>
+        <mesh filename="package://turtlebot3_description/meshes/sensors/lds.stl" scale="${0.0004*scale} ${0.0004*scale} ${0.0004*scale}"/>
       </geometry>
-      <material name="base_material"/>
     </visual>
     <collision>
@@ -48,9 +49,9 @@
     </collision>
     <inertial>
-      <mass value="0.0114" />
+      <mass value="0.1" />
       <origin xyz="0 0 0" />
-      <inertia ixx="0.001" ixy="0.0" ixz="0.0"
-               iyy="0.001" iyz="0.0"
-               izz="0.001" />
+      <inertia ixx="0.0" ixy="0.0" ixz="0.0"
+               iyy="0.0" iyz="0.0"
+               izz="0.005" />
     </inertial>
   </link>
@@ -58,22 +59,22 @@
 		<parent link="base_link" />
 		<child link="base_scan" />
-		<origin xyz="0 0 0.01905"/>
+		<origin xyz="0 0 ${0.01905*scale}"/>
 	</joint>
 	<xacro:rim_macro
 		name="left"
-		color="0.3 0 0"
-		xyz="-0.03464101615 0.02 0"
+		color="Red"
+		xyz="${-0.03464101615*scale} ${0.02*scale} 0"
 		rpy="1.570796326794896 0 1.047197551196597"
 	/>
 	<xacro:rim_macro
 		name="back"
-		color="0 0.3 0"
-		xyz="0 -0.04 0"
+		color="Green"
+		xyz="0 ${-0.04*scale} 0"
 		rpy="1.570796326794896 0 3.141592653589793"
 	/>
 	<xacro:rim_macro
 		name="right"
-		color="0 0 0.3"
-		xyz="0.03464101615 0.02 0"
+		color="Blue"
+		xyz="${0.03464101615*scale} ${0.02*scale} 0"
 		rpy="1.570796326794896 0 -1.047197551196597"
 	/>

File: localization/OpenBase/ROS/open_base/xacro/omni.gazebo.xacro (robot description, xacro)
@@ -1,5 +1,5 @@
 <?xml version="1.0"?>
 <robot name="open_base_sim" xmlns:xacro="http://ros.org/wiki/xacro">
-  <xacro:arg name="laser_visual" default="true"/>
+  <xacro:arg name="laser_visual" default="false"/>
   <xacro:arg name="imu_visual"   default="false"/>
   <!-- <gazebo>

File: localization/OpenBase/ROS/open_base/xacro/rim.urdf.xacro (robot description, xacro)
@@ -1,40 +1,41 @@
 <?xml version="1.0" ?>
 <robot xmlns:xacro="http://www.ros.org/wiki/xacro">
+	<!-- <material name="Gazebo/Red">
+		<color rgba="0.8 0.0 0.0 1.0"/>
+	</material>
+	<material name="Gazebo/Red">
+		<color rgba="0.8 0.0 0.0 1.0"/>
+	</material> -->
 	<xacro:include filename="$(find open_base)/xacro/roller.urdf.xacro"/>
-	<xacro:macro
-		name="rim_macro"
-		params="name color xyz rpy"
-	>
+	<xacro:macro name="rim_macro" params="name color xyz rpy">
+		<gazebo reference="rim_${name}_link">
+			<material>Gazebo/${color}</material>
+		</gazebo>
 		<link name="rim_${name}_link">
 			<inertial>
 				<origin xyz="0 0 -0.000343"/>
-				<mass value="0.00835758"/>
+				<mass value="0.1"/>
+				<!-- use cylinder to simulate the rim, Izz=0.5*m*r^2, Ixx=Iyy=1/12*m*(3*r^2+h^2) -->
 				<inertia
-					ixx="6.63684e-07"
+					ixx="${1/12*0.1*(3*0.101625*0.101625+0.04125*0.04125)}"
 					ixy="0"
 					ixz="0"
-					iyy="6.63684e-07"
+					iyy="${1/12*0.1*(3*0.101625*0.101625+0.04125*0.04125)}"
 					iyz="0"
-					izz="9.40333e-07"
+					izz="${0.5*0.1*0.101625*0.101625}"
 				/>
 			</inertial>
 			<visual>
 				<geometry>
-					<mesh filename="package://open_base/mesh/rim.stl"/>
+					<mesh filename="package://open_base/mesh/rim.stl" scale="${scale} ${scale} ${scale}"/>
 				</geometry>
-				<material name="rim_${name}_material">
-					<color rgba="${color} 1"/>
-				</material>
 			</visual>
 			<collision>
 				<geometry>
-					<mesh filename="package://open_base/mesh/rim.stl"/>
+					<mesh filename="package://open_base/mesh/rim.stl" scale="${scale} ${scale} ${scale}"/>
 				</geometry>
 			</collision>
 		</link>
-		<joint
-			name="rim_${name}_joint"
-			type="continuous"
-		>
+		<joint name="rim_${name}_joint" type="continuous">
 			<parent link="base_link" />
 			<child link="rim_${name}_link" />
@@ -48,5 +49,5 @@
 			parent="${name}"
 			name="e"
-			xyz="0.01355 0 0.0055"
+			xyz="${0.01355*scale} 0 ${0.0055*scale}"
 			rpy="-1.570796326794896 0 0"
 		/>
@@ -54,5 +55,5 @@
 			parent="${name}"
 			name="ne"
-			xyz="0.00958129689 0.00958129689 -0.0055"
+			xyz="${0.00958129689*scale} ${0.00958129689*scale} ${-0.0055*scale}"
 			rpy="-1.570796326794896 0 0.7853981633974483"
 		/>
@@ -60,5 +61,5 @@
 			parent="${name}"
 			name="n"
-			xyz="0 0.01355 0.0055"
+			xyz="0 ${0.01355*scale} ${0.0055*scale}"
 			rpy="-1.570796326794896 0 1.570796326794896"
 		/>
@@ -66,5 +67,5 @@
 			parent="${name}"
 			name="nw"
-			xyz="-0.00958129689 0.00958129689 -0.0055"
+			xyz="${-0.00958129689*scale} ${0.00958129689*scale} ${-0.0055*scale}"
 			rpy="-1.570796326794896 0 2.356194490192345"
 		/>
@@ -72,5 +73,5 @@
 			parent="${name}"
 			name="w"
-			xyz="-0.01355 0 0.0055"
+			xyz="${-0.01355*scale} 0 ${0.0055*scale}"
 			rpy="-1.570796326794896 0 3.141592653589793"
 		/>
@@ -78,5 +79,5 @@
 			parent="${name}"
 			name="sw"
-			xyz="-0.00958129689 -0.00958129689 -0.0055"
+			xyz="${-0.00958129689*scale} ${-0.00958129689*scale} ${-0.0055*scale}"
 			rpy="-1.570796326794896 0 -2.356194490192345"
 		/>
@@ -84,5 +85,5 @@
 			parent="${name}"
 			name="s"
-			xyz="0 -0.01355 0.0055"
+			xyz="0 ${-0.01355*scale} ${0.0055*scale}"
 			rpy="-1.570796326794896 0 -1.570796326794896"
 		/>
@@ -90,5 +91,5 @@
 			parent="${name}"
 			name="se"
-			xyz="0.00958129689 -0.00958129689 -0.0055"
+			xyz="${0.00958129689*scale} ${-0.00958129689*scale} ${-0.0055*scale}"
 			rpy="-1.570796326794896 0 -0.7853981633974483"
 		/>
@@ -96,8 +97,8 @@
 			<type>transmission_interface/SimpleTransmission</type>
 			<joint name="rim_${name}_joint">
-				<hardwareInterface>EffortJointInterface</hardwareInterface>
+				<hardwareInterface>hardware_interface/EffortJointInterface</hardwareInterface>
 			</joint>
 			<actuator name="rim_${name}_motor">
-				<hardwareInterface>EffortJointInterface</hardwareInterface>
+				<hardwareInterface>hardware_interface/EffortJointInterface</hardwareInterface>
 				<mechanicalReduction>1</mechanicalReduction>
 			</actuator>

File: localization/OpenBase/ROS/open_base/xacro/roller.urdf.xacro (robot description, xacro)
@@ -1,45 +1,44 @@
 <?xml version="1.0" ?>
 <robot xmlns:xacro="http://www.ros.org/wiki/xacro">
-	<xacro:macro
-		name="roller_macro"
-		params="parent name xyz rpy"
-	>
+	<xacro:macro name="roller_macro" params="parent name xyz rpy">
+		<gazebo reference="roller_${name}_rim_${parent}_link">
+			<material>Gazebo/Grey</material>
+			<mu>1.0</mu>
+			<mu2>1.0</mu2>
+			<kp>1e15</kp>
+			<kd>1e12</kd>
+			<minDepth>0.005</minDepth>
+			<maxVel>0.1</maxVel>
+			<fdir1>1 0 0</fdir1>
+		</gazebo>
 		<link name="roller_${name}_rim_${parent}_link">
 			<inertial>
-				<mass value="0.00113845"/>
+				<mass value="0.113845"/>
 				<inertia
-					ixx="2.53776e-08"
+					ixx="2.53776e-8"
 					ixy="0"
 					ixz="0"
-					iyy="2.53776e-08"
+					iyy="2.53776e-8"
 					iyz="0"
-					izz="1.47666e-08"
+					izz="1.47666e-8"
 				/>
 			</inertial>
 			<visual>
 				<geometry>
-					<mesh filename="package://open_base/mesh/roller.stl"/>
+					<mesh filename="package://open_base/mesh/roller.stl" scale="${scale} ${scale} ${scale}"/>
 				</geometry>
-				<material name="roller_material">
-					<color rgba="0.1 0.1 0.1 1"/>
-				</material>
 			</visual>
 			<collision>
 				<geometry>
-					<mesh filename="package://open_base/mesh/roller.stl"/>
+					<mesh filename="package://open_base/mesh/roller.stl" scale="${scale} ${scale} ${scale}"/>
 				</geometry>
 			</collision>
 		</link>
-		<joint
-			name="roller_${name}_rim_${parent}_joint"
-			type="continuous"
-		>
+		<joint name="roller_${name}_rim_${parent}_joint" type="continuous">
 			<parent link="rim_${parent}_link"/>
 			<child link="roller_${name}_rim_${parent}_link"/>
 			<axis xyz="0 0 1"/>
-			<origin
-				xyz="${xyz}"
-				rpy="${rpy}"
-			/>
+			<origin xyz="${xyz}" rpy="${rpy}"/>
+			<dynamics damping="0.0" friction="0.0001"/>
 		</joint>
 	</xacro:macro>

Commit message: Feat: basically can simulate the 3-wheeled omni robot, but when low velocity, it moves strange

File: localization/OpenBase/ROS/open_base/xacro/main.urdf.xacro (robot description, xacro)
@@ -3,5 +3,5 @@
 	<xacro:include filename="$(find open_base)/xacro/rim.urdf.xacro"/>
 	<xacro:include filename="$(find open_base)/xacro/omni.gazebo.xacro"/>
-	<xacro:property name="scale" value="7.5"/>
+	<xacro:property name="scale" value="3.0"/>
 	<gazebo reference="base_link">
 		<material>Gazebo/White</material>
@@ -13,9 +13,9 @@
 	<link name="base_link">
 		<inertial>
-      <mass value="1.0" />
+      <mass value="0.5" />
       <origin xyz="0 0 0" />
-      <inertia ixx="0.45" ixy="0.0" ixz="0.0"
-               iyy="0.45" iyz="0.0"
-               izz="0.45" />
+      <inertia ixx="0.045" ixy="0.0" ixz="0.0"
+               iyy="0.045" iyz="0.0"
+               izz="0.045" />
 		</inertial>
 		<visual>
@@ -43,5 +43,5 @@
     </visual>
     <collision>
-      <origin xyz="0.015 0 -0.0065" rpy="0 0 0"/>
+      <origin xyz="0.0 0 0.0" rpy="0 0 0"/>
       <geometry>
         <cylinder length="0.0315" radius="0.055"/>
@@ -49,5 +49,5 @@
     </collision>
     <inertial>
-      <mass value="0.1" />
+      <mass value="0.02" />
       <origin xyz="0 0 0" />
       <inertia ixx="0.0" ixy="0.0" ixz="0.0"

File: localization/OpenBase/ROS/open_base/xacro/rim.urdf.xacro (robot description, xacro)
@@ -41,8 +41,6 @@
 			<child link="rim_${name}_link" />
 			<axis xyz="0 0 1"/>
-			<origin
-				xyz="${xyz}"
-				rpy="${rpy}"
-			/>
+			<origin xyz="${xyz}" rpy="${rpy}"/>
+			<safety_controller k_position="100" k_velocity="1000" soft_lower_limit="-10" soft_upper_limit="10"/>
 		</joint>
 		<xacro:roller_macro

File: localization/OpenBase/ROS/open_base/xacro/roller.urdf.xacro (robot description, xacro)
@@ -4,11 +4,11 @@
 		<gazebo reference="roller_${name}_rim_${parent}_link">
 			<material>Gazebo/Grey</material>
-			<mu>1.0</mu>
-			<mu2>1.0</mu2>
-			<kp>1e15</kp>
-			<kd>1e12</kd>
+			<mu>1000.0</mu>
+			<mu2>0.0</mu2>
+			<kp>100</kp>
+			<kd>100</kd>
 			<minDepth>0.005</minDepth>
 			<maxVel>0.1</maxVel>
-			<fdir1>1 0 0</fdir1>
+			<fdir1>0 0 1</fdir1>
 		</gazebo>
 		<link name="roller_${name}_rim_${parent}_link">
@@ -35,5 +35,5 @@
 			</collision>
 		</link>
-		<joint name="roller_${name}_rim_${parent}_joint" type="continuous">
+		<joint name="roller_${name}_rim_${parent}_joint" type="fixed">
 			<parent link="rim_${parent}_link"/>
 			<child link="roller_${name}_rim_${parent}_link"/>

Commit message: Feat: add navigation with 3-wheeled omni robot, It can move but not that good

File: localization/OpenBase/ROS/open_base/xacro/main.urdf.xacro (robot description, xacro)
@@ -3,4 +3,5 @@
 	<xacro:include filename="$(find open_base)/xacro/rim.urdf.xacro"/>
 	<xacro:include filename="$(find open_base)/xacro/omni.gazebo.xacro"/>
+	<xacro:include filename="$(find open_base)/xacro/material.xacro"/>
 	<xacro:property name="scale" value="3.0"/>
 	<gazebo reference="base_link">
@@ -23,4 +24,5 @@
 				<mesh filename="package://open_base/mesh/base.stl" scale="${scale} ${scale} ${scale}"/>
 			</geometry>
+			<material name="White"/>
 		</visual>
 		<collision>
@@ -37,11 +39,12 @@
   <link name="base_scan">
     <visual>
-      <origin xyz="0 0 0.0" rpy="0 0 0"/>
+      <origin xyz="0 0 0" rpy="0 0 0"/>
       <geometry>
         <mesh filename="package://turtlebot3_description/meshes/sensors/lds.stl" scale="${0.0004*scale} ${0.0004*scale} ${0.0004*scale}"/>
       </geometry>
+			<material name="Brown"/>
     </visual>
     <collision>
-      <origin xyz="0.0 0 0.0" rpy="0 0 0"/>
+      <origin xyz="0.0 0 0" rpy="0 0 0"/>
       <geometry>
         <cylinder length="0.0315" radius="0.055"/>
@@ -59,5 +62,5 @@
 		<parent link="base_link" />
 		<child link="base_scan" />
-		<origin xyz="0 0 ${0.01905*scale}"/>
+		<origin xyz="0 0 ${0.03+0.01905*scale}"/>
 	</joint>
 	<xacro:rim_macro

File: localization/OpenBase/ROS/open_base/xacro/omni.gazebo.xacro (robot description, xacro)
@@ -48,5 +48,5 @@
         <range>
           <min>0.120</min>
-          <max>3.0</max>
+          <max>16.0</max>
           <resolution>0.015</resolution>
         </range>
@@ -58,5 +58,5 @@
       </ray>
       <plugin name="gazebo_ros_lds_lfcd_controller" filename="libgazebo_ros_laser.so">
-        <topicName>scan</topicName>
+        <topicName>/scan</topicName>
         <frameName>base_scan</frameName>
       </plugin>

File: localization/OpenBase/ROS/open_base/xacro/rim.urdf.xacro (robot description, xacro)
@@ -30,4 +30,5 @@
 					<mesh filename="package://open_base/mesh/rim.stl" scale="${scale} ${scale} ${scale}"/>
 				</geometry>
+				<material name="${color}"/>
 			</visual>
 			<collision>

File: localization/OpenBase/ROS/open_base/xacro/roller.urdf.xacro (robot description, xacro)
@@ -4,5 +4,5 @@
 		<gazebo reference="roller_${name}_rim_${parent}_link">
 			<material>Gazebo/Grey</material>
-			<mu>1000.0</mu>
+			<mu>0.0</mu>
 			<mu2>0.0</mu2>
 			<kp>100</kp>
@@ -28,4 +28,5 @@
 					<mesh filename="package://open_base/mesh/roller.stl" scale="${scale} ${scale} ${scale}"/>
 				</geometry>
+				<material name="Grey"/>
 			</visual>
 			<collision>
